File: doc/Schematic/BigClockSch.kicad_sch (KiCad schematic)
At the start: 8 parts

Commit message: Schematic finished, and added photos
Connections:
- no-connect marks 0 -> 1
Other:
- note added: "Buttons pulled up by arduino"
- note added: "Bypass Caps and pullup resistors omitted"
- note added: "Opt: Press - Enter Long press - Back/Menu"
- note removed: "Opt: Press - Enter Long press - Back"
- moved on the sheet: SW?

Commit message: Added PDF of Schematic
Other:
- note added: "Digits are wired in sequence of Most to Least Significant, i.e. reading order"
- note removed: "Digits are wired in sequence of Most to Least Significant"
- company: (none) -> M Chilcott
- title: (none) -> KOALA Clock
