File: doc/Schematic/LEDDigit.kicad_sch (KiCad schematic)
At the start: 24 parts

Commit message: Schematic finished, and added photos
Connections:
- net DOUT: now also D?.2 (DOUT); no longer D?.2 (DOUT)
- net +5V: now reaches D?.1 (VDD)
- net +5V: now also D?.1 (VDD), D?.1 (VDD), D?.1 (VDD), D?.1 (VDD), D?.1 (VDD), D?.1 (VDD), D?.1 (VDD), D?.1 (VDD), D?.1 (VDD), D?.1 (VDD), D?.1 (VDD), D?.1 (VDD), D?.1 (VDD), D?.1 (VDD), D?.1 (VDD), D?.1 (VDD), D?.1 (VDD), D?.1 (VDD), D?.1 (VDD), D?.1 (VDD), D?.1 (VDD), D?.1 (VDD), D?.1 (VDD)
- net GND: now reaches D?.3 (VSS)
- net GND: now also D?.3 (VSS), D?.3 (VSS), D?.3 (VSS), D?.3 (VSS), D?.3 (VSS), D?.3 (VSS), D?.3 (VSS), D?.3 (VSS), D?.3 (VSS), D?.3 (VSS), D?.3 (VSS), D?.3 (VSS), D?.3 (VSS), D?.3 (VSS), D?.3 (VSS), D?.3 (VSS), D?.3 (VSS), D?.3 (VSS), D?.3 (VSS), D?.3 (VSS), D?.3 (VSS), D?.3 (VSS), D?.3 (VSS)
- net at D?.4 (DIN): now also D?.2 (DOUT) (x12)
- net at D?.2 (DOUT): now also D?.4 (DIN) (x11)
Other:
- note added: "A"
- note added: "B"
- note added: "C"
- note added: "D"
- note added: "E"
- note added: "F"
- note added: "G"
- note added: "Numeric bit strings of form abcdefg (1 = segment on) Char Bitstring 0 1111110 1 0110000 2 1101101 3 1111001 4 0110011 5 1011011 6 1011111 7 1110000 8 1111111 9 1110011"
- note added: "Segment labels (and order)"
- note added: "Then decimal point, then colon"
- moved on the sheet: D?

Commit message: Added PDF of Schematic
Other:
- company: (none) -> M Chilcott
- title: (none) -> KOALA Clock - Digit
Changed lines of the file:
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@@
 (kicad_sch (version 20211123) (generator eeschema)
   (paper "A4")
+  (title_block
+    (title "KOALA Clock - Digit")
+    (company "M Chilcott")
+    (comment 1 "6 Identical Digits in Clock")
+  )
   (junction (at 144.78 43.18) (diameter 0) (color 0 0 0 0)
   )
